Commit message: QuadrotorX orientation

File: src/spark_softdrone/urdf/drone.urdf.xacro (robot description, xacro)
@@ -4,4 +4,5 @@
   <xacro:property name="PI" value="3.1415926535897931" />
   <xacro:property name="PI_2" value="1.5707963267948966" />
+  <xacro:property name="PI_3_4" value="2.3561944901923448" />
   <xacro:property name="PI_5_4" value="3.9269908169872414" />
     <link name="base_link"></link>
@@ -12,10 +13,10 @@
     <link name="target_cam_link"></link>
     <joint name="base_link_to_cad_link" type="fixed">
-      <origin xyz="0 0 0" rpy="0 0 -${PI_2}" />
+      <origin xyz="0 0 0" rpy="0 0 -${PI_3_4}" />
       <parent link="base_link"/>
       <child link="cad_link" />
     </joint>
     <joint name="cad_link_to_fcu_link" type="fixed">
-      <origin xyz="0.015064 -0.014986 0.064072" rpy="0 0 ${PI_2}" />
+      <origin xyz="0.015064 -0.014986 0.064072" rpy="0 0 ${PI_3_4}" />
       <parent link="cad_link"/>
       <child link="fcu_link" />

Commit message: Add nav_cam_link_tilted and corresponding joint to URDF

File: src/spark_softdrone/urdf/drone.urdf.xacro (robot description, xacro)
@@ -10,4 +10,5 @@
     <link name="fcu_link"></link>
     <link name="nav_cam_link"></link>
+    <link name="nav_cam_link_tilted"></link>
     <link name="servo_pivot_link"></link>
     <link name="target_cam_link"></link>
@@ -23,7 +24,12 @@
     </joint>
     <joint name="cad_link_to_nav_cam" type="fixed">
-      <origin xyz="-0.076587 -0.077725 0.036553" rpy="0 0.611 ${PI_5_4}" />
+      <origin xyz="-0.076587 -0.077725 0.036553" rpy="0 0 ${PI_5_4}" />
       <parent link="cad_link"/>
       <child link="nav_cam_link" />
+    </joint>
+    <joint name="nav_cam_to_nav_cam_tilted" type="fixed">
+      <origin xyz="0 0 0" rpy="0 0.611 0" />
+      <parent link="nav_cam_link"/>
+      <child link="nav_cam_link_tilted" />
     </joint>
     <joint name="cad_link_to_servo_pivot" type="revolute">

Commit message: Removed fcu_link, moved base_link to old fcu_link

File: src/spark_softdrone/urdf/drone.urdf.xacro (robot description, xacro)
@@ -8,5 +8,4 @@
     <link name="base_link"></link>
     <link name="cad_link"></link>
-    <link name="fcu_link"></link>
     <link name="nav_cam_link"></link>
     <link name="nav_cam_link_tilted"></link>
@@ -14,12 +13,7 @@
     <link name="target_cam_link"></link>
     <joint name="base_link_to_cad_link" type="fixed">
-      <origin xyz="0 0 0" rpy="0 0 -${PI_3_4}" />
+      <origin xyz="0.02123 0.0 -0.06407" rpy="0 0 -${PI_3_4}" />
       <parent link="base_link"/>
       <child link="cad_link" />
-    </joint>
-    <joint name="cad_link_to_fcu_link" type="fixed">
-      <origin xyz="0.015064 -0.014986 0.064072" rpy="0 0 ${PI_3_4}" />
-      <parent link="cad_link"/>
-      <child link="fcu_link" />
     </joint>
     <joint name="cad_link_to_nav_cam" type="fixed">

Commit message: Add mesh installation and update base_link visual in URDF

File: src/spark_softdrone/urdf/drone.urdf.xacro (robot description, xacro)
@@ -6,5 +6,15 @@
   <xacro:property name="PI_3_4" value="2.3561944901923448" />
   <xacro:property name="PI_5_4" value="3.9269908169872414" />
-    <link name="base_link"></link>
+    <link name="base_link">
+      <visual>
+        <origin xyz="0.02123 0.0 -0.06407" rpy="0 0 -${PI_3_4}" />
+        <geometry>
+          <mesh scale=".001 .001 .001" filename="package://spark_softdrone/meshes/RSISoftDroneV3.stl"/>
+        </geometry>
+        <material name="gray">
+          <color rgba="0.5 0.5 0.5 1.0"/>
+        </material>
+      </visual>
+    </link>
     <link name="cad_link"></link>
     <link name="nav_cam_link"></link>

Commit message: Update drone URDF to replace base_link visual with quadrotor model

File: src/spark_softdrone/urdf/drone.urdf.xacro (robot description, xacro)
@@ -7,5 +7,5 @@
   <xacro:property name="PI_5_4" value="3.9269908169872414" />
     <link name="base_link">
-      <visual>
+      <!-- <visual>
         <origin xyz="0.02123 0.0 -0.06407" rpy="0 0 -${PI_3_4}" />
         <geometry>
@@ -14,4 +14,14 @@
         <material name="gray">
           <color rgba="0.5 0.5 0.5 1.0"/>
+        </material>
+      </visual>
+    </link> -->
+      <visual>
+        <origin xyz="0.0 0.0 0.0" rpy="0 0 0" />
+        <geometry>
+          <mesh scale="1 1 1" filename="package://spark_softdrone/meshes/quadrotor.dae"/>
+        </geometry>
+        <material name="red">
+          <color rgba="0.7 0.3 0.3 1.0"/>
         </material>
       </visual>

Commit message: Fix t265 stuff.  Full localization pipeline to rviz on Iron working

File: src/spark_softdrone/urdf/drone.urdf.xacro (robot description, xacro)
@@ -18,5 +18,5 @@
     </link> -->
       <visual>
-        <origin xyz="0.0 0.0 0.0" rpy="0 0 0" />
+        <origin xyz="0.0 0.0 0.0" rpy="0 0 ${PI}" />
         <geometry>
           <mesh scale="1 1 1" filename="package://spark_softdrone/meshes/quadrotor.dae"/>
@@ -30,6 +30,7 @@
     <link name="nav_cam_link"></link>
     <link name="nav_cam_link_tilted"></link>
-    <link name="servo_pivot_link"></link>
-    <link name="target_cam_link"></link>
+    <!-- <link name="servo_pivot_link"></link> -->
+    <!-- <link name="target_cam_link"></link> -->
+    <link name="rgbd_cam_link"></link>
     <joint name="base_link_to_cad_link" type="fixed">
       <origin xyz="0.02123 0.0 -0.06407" rpy="0 0 -${PI_3_4}" />
@@ -47,5 +48,10 @@
       <child link="nav_cam_link_tilted" />
     </joint>
-    <joint name="cad_link_to_servo_pivot" type="revolute">
+    <joint name="cad_link_to_rgbd_cam_link" type="fixed">
+      <origin xyz="0 0.1795 -0.007" rpy="0 0.611 ${PI_2}" />
+      <parent link="cad_link"/>
+      <child link="rgbd_cam_link" />
+    </joint>
+    <!-- <joint name="cad_link_to_servo_pivot" type="revolute">
       <origin xyz="0 0.1795 -0.007" rpy="0 0.611 ${PI_2}" />
       <parent link="cad_link"/>
@@ -62,4 +68,4 @@
       <parent link="servo_pivot_link"/>
       <child link="target_cam_link" />
-    </joint>
+    </joint> -->
 </robot>

Commit message: updated urdf

File: src/spark_softdrone/urdf/drone.urdf.xacro (robot description, xacro)
@@ -32,5 +32,5 @@
     <!-- <link name="servo_pivot_link"></link> -->
     <!-- <link name="target_cam_link"></link> -->
-    <link name="rgbd_cam_link"></link>
+    <link name="camera_rgbd_link"></link>
     <joint name="base_link_to_cad_link" type="fixed">
       <origin xyz="0.02123 0.0 -0.06407" rpy="0 0 -${PI_3_4}" />
@@ -48,8 +48,8 @@
       <child link="nav_cam_link_tilted" />
     </joint>
-    <joint name="cad_link_to_rgbd_cam_link" type="fixed">
+    <joint name="cad_link_to_camera_rgbd_link" type="fixed">
       <origin xyz="0 0.1795 -0.007" rpy="0 0.611 ${PI_2}" />
       <parent link="cad_link"/>
-      <child link="rgbd_cam_link" />
+      <child link="camera_rgbd_link" />
     </joint>
     <!-- <joint name="cad_link_to_servo_pivot" type="revolute">
